File: myRIO/Demo Board/myRIODemoBoard.sch (KiCad schematic (older format))
At the start: 5 parts

Commit message: Complete PCB. Needs Review.
Parts:
- gave numbers to parts that had none: 2
- renumbered 7SEG to 7SEG1
Changed lines of the file:
@@
 $EndDescr
 $Comp
-L MXP U?
+L MXP U1
 U 1 1 53079AD1
 P 5700 3800
-F 0 "U?" H 6250 2800 60  0000 C CNN
+F 0 "U1" H 6250 2800 60  0000 C CNN
 F 1 "MXP" H 5750 4750 60  0000 C CNN
 F 2 "~" H 5800 3900 60  0000 C CNN
@@
 $EndComp
 $Comp
-L GND #PWR?
+L GND #PWR01
 U 1 1 5307ADAC
 P 4400 6150
-F 0 "#PWR?" H 4400 6150 30  0001 C CNN
+F 0 "#PWR01" H 4400 6150 30  0001 C CNN
 F 1 "GND" H 4400 6080 30  0001 C CNN
 F 2 "" H 4400 6150 60  0000 C CNN
@@
 $EndComp
 $Comp
-L POT RV?
+L POT RV1
 U 1 1 5307AE6F
 P 7650 4400
-F 0 "RV?" H 7650 4300 50  0000 C CNN
+F 0 "RV1" H 7650 4300 50  0000 C CNN
 F 1 "POT" H 7650 4400 50  0000 C CNN
 F 2 "~" H 7650 4400 60  0000 C CNN
@@
 $EndComp
 $Comp
-L +5V #PWR?
+L +5V #PWR02
 U 1 1 5307B1A6
 P 7650 4050
-F 0 "#PWR?" H 7650 4140 20  0001 C CNN
+F 0 "#PWR02" H 7650 4140 20  0001 C CNN
 F 1 "+5V" H 7650 4140 30  0000 C CNN
 F 2 "" H 7650 4050 60  0000 C CNN
@@
 $EndComp
 $Comp
-L +5V #PWR?
+L +5V #PWR03
 U 1 1 5307B303
 P 6750 4750
-F 0 "#PWR?" H 6750 4840 20  0001 C CNN
+F 0 "#PWR03" H 6750 4840 20  0001 C CNN
 F 1 "+5V" H 6750 4840 30  0000 C CNN
 F 2 "" H 6750 4750 60  0000 C CNN
@@
 $EndComp
 $Comp
-L 7SEGMENTS 7SEG
+L 7SEGMENTS 7SEG1
 U 1 1 5307B582
 P 6200 2000
-F 0 "7SEG" H 6200 2550 60  0000 C CNN
+F 0 "7SEG1" H 6200 2550 60  0000 C CNN
 F 1 "7SEGMENTS" H 6200 1550 60  0000 C CNN
 F 2 "" H 6200 2000 60  0000 C CNN
@@
 $EndComp
 $Comp
-L +3.3V #PWR?
+L +3.3V #PWR04
 U 1 1 5307B65C
 P 6750 2950
-F 0 "#PWR?" H 6750 2910 30  0001 C CNN
+F 0 "#PWR04" H 6750 2910 30  0001 C CNN
 F 1 "+3.3V" H 6750 3060 30  0000 C CNN
 F 2 "" H 6750 2950 60  0000 C CNN
@@
 $EndComp
 $Comp
-L +3.3V #PWR?
+L +3.3V #PWR05
 U 1 1 5307B712
 P 5500 1450
-F 0 "#PWR?" H 5500 1410 30  0001 C CNN
+F 0 "#PWR05" H 5500 1410 30  0001 C CNN
 F 1 "+3.3V" H 5500 1560 30  0000 C CNN
 F 2 "" H 5500 1450 60  0000 C CNN
@@
 	7650 6050 4400 6050
 $Comp
-L GND #PWR?
+L GND #PWR06
 U 1 1 5307C168
 P 4100 4650
-F 0 "#PWR?" H 4100 4650 30  0001 C CNN
+F 0 "#PWR06" H 4100 4650 30  0001 C CNN
 F 1 "GND" H 4100 4580 30  0001 C CNN
 F 2 "" H 4100 4650 60  0000 C CNN

Commit message: Small updates to footprints, schematic, etc.
Connections:
- net a: now reaches 7SEG1.7 (a), U1.11 (DIO0)
- net b: now reaches 7SEG1.6 (b), U1.13 (DIO1)
- net c: now reaches 7SEG1.4 (c), U1.15 (DIO2)
- net d: now reaches 7SEG1.2 (d), U1.17 (DIO3)
- net e: now reaches 7SEG1.1 (e), U1.19 (DIO4)
- net f: now reaches 7SEG1.9 (f), U1.21 (DIO5/SPI.CLK)
- net g: now reaches 7SEG1.10 (g), U1.23 (DIO6/SPI.MISO)
- net dp: now reaches 7SEG1.5 (DP), U1.25 (DIO7/SPI.MOSI)
Changed lines of the file:
@@
 Sheet 1 1
 Title ""
-Date "21 feb 2014"
+Date "24 feb 2014"
 Rev ""
 Comp ""
@@
 Connection ~ 5500 1550
 Wire Wire Line
-	6800 2200 7100 2200
+	6800 2200 7500 2200
 Wire Wire Line
 	6650 3500 7100 3500
@@
 	7400 4100 7400 1600
 Wire Wire Line
-	7400 1600 6800 1600
-Wire Wire Line
-	6800 1700 7350 1700
+	6800 1600 7500 1600
+Wire Wire Line
+	6800 1700 7650 1700
 Wire Wire Line
 	7350 1700 7350 4000
 Wire Wire Line
-	6800 1800 7300 1800
+	6800 1800 7500 1800
 Wire Wire Line
 	7300 1800 7300 3900
@@
 	7250 3800 7250 1900
 Wire Wire Line
-	7250 1900 6800 1900
-Wire Wire Line
-	6800 2000 7200 2000
+	6800 1900 7650 1900
+Wire Wire Line
+	6800 2000 7500 2000
 Wire Wire Line
 	7200 2000 7200 3700
@@
 	7150 3600 7150 2100
 Wire Wire Line
-	7150 2100 6800 2100
+	6800 2100 7650 2100
 Wire Wire Line
 	7350 4000 6650 4000
@@
 	5500 1550 5600 1550
 Wire Wire Line
-	5600 2250 5500 2250
+	5400 2250 5600 2250
 Wire Wire Line
 	5500 2250 5500 2650
@@
 	4750 3200 4600 3200
 Connection ~ 4600 3300
+Text GLabel 7500 1600 2    60   Input ~ 0
+a
+Connection ~ 7400 1600
+Text GLabel 7650 1700 2    60   Input ~ 0
+b
+Text GLabel 7500 1800 2    60   Input ~ 0
+c
+Connection ~ 7350 1700
+Connection ~ 7300 1800
+Text GLabel 7500 2000 2    60   Input ~ 0
+e
+Text GLabel 7650 1900 2    60   Input ~ 0
+d
+Text GLabel 7500 2200 2    60   Input ~ 0
+g
+Text GLabel 7650 2100 2    60   Input ~ 0
+f
+Connection ~ 7100 2200
+Connection ~ 7150 2100
+Connection ~ 7200 2000
+Connection ~ 7250 1900
+Text GLabel 5400 2250 0    60   Input ~ 0
+dp
+Connection ~ 5500 2250
 $EndSCHEMATC

Commit message: Prototype Order of Rev 1.0
Parts:
- 7SEG1: value 7SEGMENTS -> 7-Segment Display
- RV1: value POT -> Potentiometer
- U1: value MXP -> myRIO MXP
Connections:
- net +3.3V: now also RV1.3
- net +5V: no longer RV1.3
Changed lines of the file:
@@
 Sheet 1 1
 Title ""
-Date "24 feb 2014"
+Date "25 feb 2014"
 Rev ""
 Comp ""
@@
 P 5700 3800
 F 0 "U1" H 6250 2800 60  0000 C CNN
-F 1 "MXP" H 5750 4750 60  0000 C CNN
+F 1 "myRIO MXP" H 5750 4750 60  0000 C CNN
 F 2 "~" H 5800 3900 60  0000 C CNN
 F 3 "~" H 5800 3900 60  0000 C CNN
@@
 P 7650 4400
 F 0 "RV1" H 7650 4300 50  0000 C CNN
-F 1 "POT" H 7650 4400 50  0000 C CNN
+F 1 "Potentiometer" H 7650 4200 50  0000 C CNN
 F 2 "~" H 7650 4400 60  0000 C CNN
 F 3 "~" H 7650 4400 60  0000 C CNN
@@
 $Comp
 L +5V #PWR02
-U 1 1 5307B1A6
-P 7650 4050
-F 0 "#PWR02" H 7650 4140 20  0001 C CNN
-F 1 "+5V" H 7650 4140 30  0000 C CNN
-F 2 "" H 7650 4050 60  0000 C CNN
-F 3 "" H 7650 4050 60  0000 C CNN
-	1    7650 4050
-	1    0    0    -1
-$EndComp
-$Comp
-L +5V #PWR03
 U 1 1 5307B303
 P 6750 4750
-F 0 "#PWR03" H 6750 4840 20  0001 C CNN
+F 0 "#PWR02" H 6750 4840 20  0001 C CNN
 F 1 "+5V" H 6750 4840 30  0000 C CNN
 F 2 "" H 6750 4750 60  0000 C CNN
@@
 P 6200 2000
 F 0 "7SEG1" H 6200 2550 60  0000 C CNN
-F 1 "7SEGMENTS" H 6200 1550 60  0000 C CNN
+F 1 "7-Segment Display" H 6200 1550 60  0000 C CNN
 F 2 "" H 6200 2000 60  0000 C CNN
 F 3 "" H 6200 2000 60  0000 C CNN
@@
 $EndComp
 $Comp
-L +3.3V #PWR04
+L +3.3V #PWR03
 U 1 1 5307B65C
 P 6750 2950
-F 0 "#PWR04" H 6750 2910 30  0001 C CNN
+F 0 "#PWR03" H 6750 2910 30  0001 C CNN
 F 1 "+3.3V" H 6750 3060 30  0000 C CNN
 F 2 "" H 6750 2950 60  0000 C CNN
@@
 $EndComp
 $Comp
-L +3.3V #PWR05
+L +3.3V #PWR04
 U 1 1 5307B712
 P 5500 1450
-F 0 "#PWR05" H 5500 1410 30  0001 C CNN
+F 0 "#PWR04" H 5500 1410 30  0001 C CNN
 F 1 "+3.3V" H 5500 1560 30  0000 C CNN
 F 2 "" H 5500 1450 60  0000 C CNN
@@
 	6900 4500 6650 4500
 Wire Wire Line
-	7650 4050 7650 4150
-Wire Wire Line
 	7500 4400 6650 4400
 Wire Wire Line
@@
 	7650 6050 4400 6050
 $Comp
-L GND #PWR06
+L GND #PWR05
 U 1 1 5307C168
 P 4100 4650
-F 0 "#PWR06" H 4100 4650 30  0001 C CNN
+F 0 "#PWR05" H 4100 4650 30  0001 C CNN
 F 1 "GND" H 4100 4580 30  0001 C CNN
 F 2 "" H 4100 4650 60  0000 C CNN
@@
 dp
 Connection ~ 5500 2250
+$Comp
+L +3.3V #PWR06
+U 1 1 530CD111
+P 7650 4050
+F 0 "#PWR06" H 7650 4010 30  0001 C CNN
+F 1 "+3.3V" H 7650 4160 30  0000 C CNN
+F 2 "" H 7650 4050 60  0000 C CNN
+F 3 "" H 7650 4050 60  0000 C CNN
+	1    7650 4050
+	1    0    0    -1
+$EndComp
+Wire Wire Line
+	7650 4050 7650 4150
 $EndSCHEMATC

Commit message: Updated myRIO Demo Board to Rev 1.1. Modified component IDs for manufacturing. Adjusted silk screen.
Parts:
- renumbered U1 to MXP1, 7SEG1 to SEV_SEG1
Changed lines of the file:
@@
 Sheet 1 1
 Title ""
-Date "25 feb 2014"
+Date "3 mar 2014"
 Rev ""
 Comp ""
@@
 $EndDescr
 $Comp
-L MXP U1
+L MXP MXP1
 U 1 1 53079AD1
 P 5700 3800
-F 0 "U1" H 6250 2800 60  0000 C CNN
+F 0 "MXP1" H 6250 2800 60  0000 C CNN
 F 1 "myRIO MXP" H 5750 4750 60  0000 C CNN
 F 2 "~" H 5800 3900 60  0000 C CNN
@@
 $EndComp
 $Comp
-L 7SEGMENTS 7SEG1
+L 7SEGMENTS SEV_SEG1
 U 1 1 5307B582
 P 6200 2000
-F 0 "7SEG1" H 6200 2550 60  0000 C CNN
+F 0 "SEV_SEG1" H 6200 2550 60  0000 C CNN
 F 1 "7-Segment Display" H 6200 1550 60  0000 C CNN
 F 2 "" H 6200 2000 60  0000 C CNN

Commit message: Updated BOM and component IDs to work better with Screaming Circuits  parser
Parts:
- renumbered SEV_SEG1 to SEG1
Changed lines of the file:
@@
 $EndComp
 $Comp
-L 7SEGMENTS SEV_SEG1
+L 7SEGMENTS SEG1
 U 1 1 5307B582
 P 6200 2000
-F 0 "SEV_SEG1" H 6200 2550 60  0000 C CNN
+F 0 "SEG1" H 6200 2550 60  0000 C CNN
 F 1 "7-Segment Display" H 6200 1550 60  0000 C CNN
 F 2 "" H 6200 2000 60  0000 C CNN

Commit message: Updated R1 to 200k in schematic, BOM and silkscreen Generated new gerbers.
Parts:
- R1: value 1k -> 200k
Changed lines of the file:
@@
 Sheet 1 1
 Title ""
-Date "3 mar 2014"
+Date "7 apr 2014"
 Rev ""
 Comp ""
@@
 P 4400 5100
 F 0 "R1" V 4480 5100 40  0000 C CNN
-F 1 "1k" V 4407 5101 40  0000 C CNN
+F 1 "200k" V 4407 5101 40  0000 C CNN
 F 2 "~" V 4330 5100 30  0000 C CNN
 F 3 "~" H 4400 5100 30  0000 C CNN
